File: schematic/UniversalboxArm1-0.kicad_pcb (KiCad board)
At the start: 4 copper layers, 112 x 57 mm, 170 parts, among them J1 USB_B_Micro, J110 Conn_01x03_Male, J120 Conn_02x04_Counter_Clockwise, J121 Conn_01x02_Male, J20 AVR-ISP-6, J50 Conn_01x14_Female, J60 Conn_01x06_Female, J61 Conn_02x08_Odd_Even, J62 Conn_02x04_Odd_Even, J90 Conn_02x03_Odd_Even, J91 Conn_02x04_Odd_Even, K90 IM01, K91 IM01, K92 IM01, K93 IM01, Q120 IRLML6402, Q20 BCX56-16, Q21 BSS138, Q22 BSS138, Q23 IRLML6402, Q24 IRLML6402, Q25 BSS138, Q50 IRLML6402, Q51 IRLML6402, Q60 BSS138, Q61 BSS138, Q62 BSS138, Q90 BSS138, Q91 BSS138, Q92 BSS138, Q93 BSS138, SW60 SW_SPST, SW61 SW_SPST, SW62 SW_SPST, SW63 SW_SPST, U1 USBLC6-2SC6, U110 MAX3221, U130 TSOP312xx, U2 LP38693MP-3.3, U20 ATtiny861A-SU, U21 REF3020, U22 MCP6542, U50 AT45DB641-S, U60 STM32L452RETx, U61 MCP65R41T-1202E, Y60 32768Hz, Y61 8MHz

Commit message: Schematic: Revision 0.9 Add worarounds for electric issues when the internal bootloader is active - bug 10. Document bug 11 - wrong signal names on PCB
Connections:
- net /Led2Red renamed /Led1Red
- net /Led2green renamed /Led1green
Changed lines of the file:
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@@
   (title_block
     (title UniversalboxArm)
-    (date 2022-01-17)
-    (rev 0.8)
+    (date 2022-02-20)
+    (rev 0.9)
     (company "Malte Marwedel")
   )
@@
   (net 153 /KeyUp)
   (net 154 /KeyDown)
-  (net 155 /Led2green)
-  (net 156 /Led2Red)
-  (net 157 /AvrOutResetArm)
+  (net 155 /AvrOutResetArm)
+  (net 156 /Led1green)
+  (net 157 /Led1Red)
   (net_class Default "Dies ist die voreingestellte Netzklasse."
     (clearance 0.25)
@@
     (add_net /LcdA0)
     (add_net /LcdCs)
-    (add_net /Led2Red)
-    (add_net /Led2green)
+    (add_net /Led1Red)
+    (add_net /Led1green)
     (add_net /Motor1F)
     (add_net /Motor1R)
@@
       (net 152 /KeyRight))
     (pad 61 smd rect (at -2.25 -5.9 270) (size 1.4 0.25) (layers F.Cu F.Paste F.Mask)
-      (net 156 /Led2Red))
+      (net 157 /Led1Red))
     (pad 60 smd rect (at -1.75 -5.9 270) (size 1.4 0.25) (layers F.Cu F.Paste F.Mask)
       (net 130 "Net-(R71-Pad1)"))
@@
       (net 100 /SwDo_Spi1Sck))
     (pad 54 smd rect (at 1.25 -5.9 270) (size 1.4 0.25) (layers F.Cu F.Paste F.Mask)
-      (net 155 /Led2green))
+      (net 156 /Led1green))
     (pad 53 smd rect (at 1.75 -5.9 270) (size 1.4 0.25) (layers F.Cu F.Paste F.Mask)
       (net 72 /SpiAvrDi))
@@
     )
     (pad 2 smd roundrect (at 1.025 0 90) (size 1.15 1.4) (layers F.Cu F.Paste F.Mask) (roundrect_rratio 0.2173904347826087)
-      (net 156 /Led2Red))
+      (net 157 /Led1Red))
     (pad 1 smd roundrect (at -1.025 0 90) (size 1.15 1.4) (layers F.Cu F.Paste F.Mask) (roundrect_rratio 0.2173904347826087)
       (net 47 "Net-(D61-Pad1)"))
@@
       (net 48 "Net-(D61-Pad3)"))
     (pad 2 smd roundrect (at 1.025 0 90) (size 1.15 1.4) (layers F.Cu F.Paste F.Mask) (roundrect_rratio 0.2173904347826087)
-      (net 155 /Led2green))
+      (net 156 /Led1green))
     (model ${KISYS3DMOD}/Resistor_SMD.3dshapes/R_0805_2012Metric.wrl
       (at (xyz 0 0 0))
@@
     )
     (pad 1 smd rect (at -1 -0.95) (size 0.9 0.8) (layers F.Cu F.Paste F.Mask)
-      (net 157 /AvrOutResetArm))
+      (net 155 /AvrOutResetArm))
     (pad 2 smd rect (at -1 0.95) (size 0.9 0.8) (layers F.Cu F.Paste F.Mask)
       (net 3 GND))
@@
       (net 3 GND))
     (pad 1 smd roundrect (at -1.025 0 90) (size 1.15 1.4) (layers F.Cu F.Paste F.Mask) (roundrect_rratio 0.2173904347826087)
-      (net 157 /AvrOutResetArm))
+      (net 155 /AvrOutResetArm))
     (model ${KISYS3DMOD}/Resistor_SMD.3dshapes/R_0805_2012Metric.wrl
       (at (xyz 0 0 0))
@@
       (net 39 "Net-(J20-Pad5)"))
     (pad 11 smd rect (at 4.7 5.715) (size 1.95 0.6) (layers F.Cu F.Paste F.Mask)
-      (net 157 /AvrOutResetArm))
+      (net 155 /AvrOutResetArm))
     (pad 12 smd rect (at 4.7 4.445) (size 1.95 0.6) (layers F.Cu F.Paste F.Mask)
       (net 24 "Net-(R23-Pad1)"))
@@
   (segment (start 177.3 108.7) (end 176.75 109.25) (width 0.5) (layer F.Cu) (net 35))
   (via (at 176.75 109.25) (size 0.8) (drill 0.4) (layers F.Cu B.Cu) (net 35))
-  (segment (start 155 104.6) (end 149.367839 104.6) (width 0.5) (layer F.Cu) (net 157))
-  (segment (start 143.638612 103.611404) (end 142.750016 104.5) (width 0.5) (layer F.Cu) (net 157))
-  (segment (start 145.411406 103.611404) (end 143.638612 103.611404) (width 0.5) (layer F.Cu) (net 157))
-  (segment (start 146.549999 105.300001) (end 146.549999 104.749997) (width 0.5) (layer F.Cu) (net 157))
-  (segment (start 146.549999 104.749997) (end 145.411406 103.611404) (width 0.5) (layer F.Cu) (net 157))
-  (segment (start 146.649999 105.400001) (end 146.549999 105.300001) (width 0.5) (layer F.Cu) (net 157))
-  (segment (start 148.567838 105.400001) (end 146.649999 105.400001) (width 0.5) (layer F.Cu) (net 157))
-  (segment (start 149.367839 104.6) (end 148.567838 105.400001) (width 0.5) (layer F.Cu) (net 157))
-  (segment (start 140.25 106.8) (end 140.75 106.3) (width 0.5) (layer F.Cu) (net 157))
-  (segment (start 137 106.8) (end 140.25 106.8) (width 0.5) (layer F.Cu) (net 157))
-  (segment (start 140.950016 106.3) (end 143.638612 103.611404) (width 0.5) (layer F.Cu) (net 157))
-  (segment (start 140.75 106.3) (end 140.950016 106.3) (width 0.5) (layer F.Cu) (net 157))
   (segment (start 137.060001 97.849999) (end 137 97.91) (width 0.5) (layer F.Cu) (net 36))
   (segment (start 150.54 95.6) (end 150.765 95.825) (width 0.5) (layer F.Cu) (net 36))
@@
   (segment (start 160.75 77.5) (end 161 77.25) (width 0.25) (layer B.Cu) (net 154))
   (segment (start 159.75 77.5) (end 160.75 77.5) (width 0.25) (layer B.Cu) (net 154))
-  (via (at 154.25 85.5) (size 0.8) (drill 0.4) (layers F.Cu B.Cu) (net 155))
-  (segment (start 154.75 85) (end 154.25 85.5) (width 0.25) (layer F.Cu) (net 155))
-  (segment (start 154.75 82.2) (end 154.75 85) (width 0.25) (layer F.Cu) (net 155))
-  (segment (start 155.088594 95.607165) (end 158.481429 99) (width 0.5) (layer B.Cu) (net 155))
-  (segment (start 155.088594 91.588594) (end 155.088594 95.607165) (width 0.5) (layer B.Cu) (net 155))
-  (segment (start 154.25 90.75) (end 155.088594 91.588594) (width 0.5) (layer B.Cu) (net 155))
-  (segment (start 158.481429 99) (end 159.75 99) (width 0.5) (layer B.Cu) (net 155))
-  (segment (start 154.25 85.5) (end 154.25 90.75) (width 0.5) (layer B.Cu) (net 155))
-  (segment (start 161.4 98.75) (end 161.15 99) (width 0.5) (layer F.Cu) (net 155))
-  (segment (start 160.315685 99) (end 159.75 99) (width 0.5) (layer F.Cu) (net 155))
-  (segment (start 161.15 99) (end 160.315685 99) (width 0.5) (layer F.Cu) (net 155))
-  (via (at 159.75 99) (size 0.8) (drill 0.4) (layers F.Cu B.Cu) (net 155))
-  (via (at 158.25 84.25) (size 0.8) (drill 0.4) (layers F.Cu B.Cu) (net 156))
-  (segment (start 158.2 84.2) (end 158.25 84.25) (width 0.25) (layer F.Cu) (net 156))
-  (segment (start 158.25 82.2) (end 158.25 84.2) (width 0.25) (layer F.Cu) (net 156))
-  (via (at 163.75 97.25) (size 0.8) (drill 0.4) (layers F.Cu B.Cu) (net 156))
-  (segment (start 158.25 84.25) (end 158.25 89.75) (width 0.5) (layer B.Cu) (net 156))
-  (segment (start 163.75 98.95) (end 163.75 97.25) (width 0.5) (layer F.Cu) (net 156))
-  (segment (start 158.25 89.75) (end 159.75 91.25) (width 0.5) (layer B.Cu) (net 156))
-  (segment (start 159.75 91.25) (end 160.482 91.25) (width 0.5) (layer B.Cu) (net 156))
-  (segment (start 160.482 91.25) (end 163.75 94.518) (width 0.5) (layer B.Cu) (net 156))
-  (segment (start 163.75 94.518) (end 163.75 97.25) (width 0.5) (layer B.Cu) (net 156))
+  (segment (start 155 104.6) (end 149.367839 104.6) (width 0.5) (layer F.Cu) (net 155))
+  (segment (start 143.638612 103.611404) (end 142.750016 104.5) (width 0.5) (layer F.Cu) (net 155))
+  (segment (start 145.411406 103.611404) (end 143.638612 103.611404) (width 0.5) (layer F.Cu) (net 155))
+  (segment (start 146.549999 105.300001) (end 146.549999 104.749997) (width 0.5) (layer F.Cu) (net 155))
+  (segment (start 146.549999 104.749997) (end 145.411406 103.611404) (width 0.5) (layer F.Cu) (net 155))
+  (segment (start 146.649999 105.400001) (end 146.549999 105.300001) (width 0.5) (layer F.Cu) (net 155))
+  (segment (start 148.567838 105.400001) (end 146.649999 105.400001) (width 0.5) (layer F.Cu) (net 155))
+  (segment (start 149.367839 104.6) (end 148.567838 105.400001) (width 0.5) (layer F.Cu) (net 155))
+  (segment (start 140.25 106.8) (end 140.75 106.3) (width 0.5) (layer F.Cu) (net 155))
+  (segment (start 137 106.8) (end 140.25 106.8) (width 0.5) (layer F.Cu) (net 155))
+  (segment (start 140.950016 106.3) (end 143.638612 103.611404) (width 0.5) (layer F.Cu) (net 155))
+  (segment (start 140.75 106.3) (end 140.950016 106.3) (width 0.5) (layer F.Cu) (net 155))
+  (via (at 154.25 85.5) (size 0.8) (drill 0.4) (layers F.Cu B.Cu) (net 156))
+  (segment (start 154.75 85) (end 154.25 85.5) (width 0.25) (layer F.Cu) (net 156))
+  (segment (start 154.75 82.2) (end 154.75 85) (width 0.25) (layer F.Cu) (net 156))
+  (segment (start 155.088594 95.607165) (end 158.481429 99) (width 0.5) (layer B.Cu) (net 156))
+  (segment (start 155.088594 91.588594) (end 155.088594 95.607165) (width 0.5) (layer B.Cu) (net 156))
+  (segment (start 154.25 90.75) (end 155.088594 91.588594) (width 0.5) (layer B.Cu) (net 156))
+  (segment (start 158.481429 99) (end 159.75 99) (width 0.5) (layer B.Cu) (net 156))
+  (segment (start 154.25 85.5) (end 154.25 90.75) (width 0.5) (layer B.Cu) (net 156))
+  (segment (start 161.4 98.75) (end 161.15 99) (width 0.5) (layer F.Cu) (net 156))
+  (segment (start 160.315685 99) (end 159.75 99) (width 0.5) (layer F.Cu) (net 156))
+  (segment (start 161.15 99) (end 160.315685 99) (width 0.5) (layer F.Cu) (net 156))
+  (via (at 159.75 99) (size 0.8) (drill 0.4) (layers F.Cu B.Cu) (net 156))
+  (via (at 158.25 84.25) (size 0.8) (drill 0.4) (layers F.Cu B.Cu) (net 157))
+  (segment (start 158.2 84.2) (end 158.25 84.25) (width 0.25) (layer F.Cu) (net 157))
+  (segment (start 158.25 82.2) (end 158.25 84.2) (width 0.25) (layer F.Cu) (net 157))
+  (via (at 163.75 97.25) (size 0.8) (drill 0.4) (layers F.Cu B.Cu) (net 157))
+  (segment (start 158.25 84.25) (end 158.25 89.75) (width 0.5) (layer B.Cu) (net 157))
+  (segment (start 163.75 98.95) (end 163.75 97.25) (width 0.5) (layer F.Cu) (net 157))
+  (segment (start 158.25 89.75) (end 159.75 91.25) (width 0.5) (layer B.Cu) (net 157))
+  (segment (start 159.75 91.25) (end 160.482 91.25) (width 0.5) (layer B.Cu) (net 157))
+  (segment (start 160.482 91.25) (end 163.75 94.518) (width 0.5) (layer B.Cu) (net 157))
+  (segment (start 163.75 94.518) (end 163.75 97.25) (width 0.5) (layer B.Cu) (net 157))
   (zone (net 74) (net_name /ShieldGND) (layer F.Cu) (hatch edge 0.508)
     (priority 1)

Commit message: Schematic: Version 0.11, update parts, reroute LCD reset
LCD reset is now connected to PC2, this allows I2C on PC0 and PC1 to be used.
R34 has been reduced to 470Ohm.
Q61 and Q62 are replaced by IRLML6344 to switch higher currents.
R55 has been added. This should allow to access the flash with 4MHz instead of 250kHz.

Measurements on R55 show the required low level of 1V is now reached within 250ns.
Parts:
- Q61, Q62: value BSS138 -> IRLML6344
- R34: value 1kΩ -> 470Ω

Commit message: Schematic: Fix power surge of ESP-01 module
Add C121, reduce C120. Make C4 not recommend.
Schematic vesion 0.12.
Parts:
- C120: value 100µF -> 4.7µF
